File: test board.sch (KiCad schematic (older format))
At the start: 129 parts, among them J1 Conn_01x02, J10 Conn_01x02, J11 Conn_01x02, J12 Conn_01x02, J13 Conn_01x02, J14 Conn_01x02, J15 Conn_01x02, J16 Conn_01x02, J17 Conn_01x02, J18 Conn_01x02, J19 Conn_01x02, J2 Conn_01x02, J20 Conn_01x02, J21 Conn_01x02, J22 Conn_01x02, J23 Conn_01x07, J24 Conn_01x07, J25 Conn_01x01, J26 Conn_01x01, J3 Conn_01x02, J4 Conn_01x02, J5 Conn_01x02, J6 Conn_01x02, J7 Conn_01x02, J8 Conn_01x02, J9 Conn_01x02, T1 Transformer_1P_1S, T2 Transformer_1P_1S, U1 LM5180QNGURQ1, U2 LM5180QNGURQ1

Commit message: more edits to schematic and began laying out pcb
Parts:
- removed LOGO3: Logo_Placeholder, UTSVT_Special:Aro, symbol utsvt-misc:Logo_Placeholder
- C10, C2, C3, C4, C5, C6, C7, C8, C9: value 500u -> 6.8u
- LOGO1: value Logo_Placeholder -> Hallock
- LOGO2: value Logo_Placeholder -> UTSVT_Logo
Connections:
- net at D4.2 (A), RV1.2, T1.2 (AB)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: no longer RV1.1
- net at D3.2 (A), RV2.2, T2.2 (AB)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: no longer RV2.1
- net GNDREF: no longer names the net of C13.2, J13.2 (Pin_2), T2.3 (SA), TP19.1
- net GNDREF: no longer C14.2, J12.2 (Pin_2), T1.3 (SA), TP17.1
- new net: C14.2, J12.2 (Pin_2), T1.3 (SA), TP17.1
- no-connect marks 6 -> 8
Other:
- moved on the sheet: TP13, TP15
Changed lines of the file:
@@
 Wire Wire Line
 	15950 9750 16450 9750
-Wire Wire Line
-	16600 9550 16550 9550
-Wire Wire Line
-	16000 9550 16000 9350
 Connection ~ 16000 9350
 Wire Wire Line
 	16000 9350 16040 9350
 Wire Wire Line
-	16600 9550 16800 9550
-Wire Wire Line
-	16800 9550 16800 9700
-Wire Wire Line
 	16800 9700 16750 9700
-Connection ~ 16600 9550
 $Comp
 L Connector:TestPoint TP13
 U 1 1 5FEE414A
-P 16550 9550
-F 0 "TP13" H 16608 9668 50  0000 L CNN
-F 1 "Pot1-TestPoint1" H 16608 9577 50  0000 L CNN
-F 2 "TestPoint:TestPoint_Keystone_5005-5009_Compact" H 16750 9550 50  0001 C CNN
-F 3 "~" H 16750 9550 50  0001 C CNN
-	1    16550 9550
-	1    0    0    -1
-$EndComp
-Connection ~ 16550 9550
-Wire Wire Line
-	16550 9550 16000 9550
+P 16800 9450
+F 0 "TP13" V 16950 9700 50  0000 L CNN
+F 1 "Pot1-TestPoint1" V 16858 9477 50  0000 L CNN
+F 2 "TestPoint:TestPoint_Keystone_5005-5009_Compact" H 17000 9450 50  0001 C CNN
+F 3 "~" H 17000 9450 50  0001 C CNN
+	1    16800 9450
+	0    1    1    0
+$EndComp
 $Comp
 L Connector:TestPoint TP14
@@
 P 8850 4250
 F 0 "C2" H 8965 4296 50  0000 L CNN
-F 1 "500u" H 8965 4205 50  0000 L CNN
+F 1 "6.8u" H 8965 4205 50  0000 L CNN
 F 2 "Capacitor_SMD:C_0805_2012Metric" H 8888 4100 50  0001 C CNN
 F 3 "~" H 8850 4250 50  0001 C CNN
@@
 	15950 11900 16450 11900
 Wire Wire Line
-	16600 11700 16550 11700
-Wire Wire Line
-	16000 11700 16000 11500
-Wire Wire Line
-	16600 11700 16800 11700
-Wire Wire Line
-	16800 11700 16800 11850
-Wire Wire Line
 	16800 11850 16750 11850
-Connection ~ 16600 11700
 $Comp
 L Connector:TestPoint TP15
 U 1 1 609BF60F
-P 16550 11700
-F 0 "TP15" H 16800 11850 50  0000 L CNN
-F 1 "Pot2-TestPoint1" H 16650 11750 50  0000 L CNN
-F 2 "TestPoint:TestPoint_Keystone_5005-5009_Compact" H 16750 11700 50  0001 C CNN
-F 3 "~" H 16750 11700 50  0001 C CNN
-	1    16550 11700
-	1    0    0    -1
-$EndComp
-Connection ~ 16550 11700
-Wire Wire Line
-	16550 11700 16000 11700
+P 16800 11650
+F 0 "TP15" V 16800 12000 50  0000 L CNN
+F 1 "Pot2-TestPoint1" V 16700 11750 50  0000 L CNN
+F 2 "TestPoint:TestPoint_Keystone_5005-5009_Compact" H 17000 11650 50  0001 C CNN
+F 3 "~" H 17000 11650 50  0001 C CNN
+	1    16800 11650
+	0    1    1    0
+$EndComp
 Connection ~ 16000 11500
 Wire Wire Line
@@
 P 8850 5050
 F 0 "C3" H 8965 5096 50  0000 L CNN
-F 1 "500u" H 8965 5005 50  0000 L CNN
+F 1 "6.8u" H 8965 5005 50  0000 L CNN
 F 2 "Capacitor_SMD:C_0805_2012Metric" H 8888 4900 50  0001 C CNN
 F 3 "~" H 8850 5050 50  0001 C CNN
@@
 P 8850 5850
 F 0 "C4" H 8965 5896 50  0000 L CNN
-F 1 "500u" H 8965 5805 50  0000 L CNN
+F 1 "6.8u" H 8965 5805 50  0000 L CNN
 F 2 "Capacitor_SMD:C_0805_2012Metric" H 8888 5700 50  0001 C CNN
 F 3 "~" H 8850 5850 50  0001 C CNN
@@
 P 8850 6650
 F 0 "C5" H 8965 6696 50  0000 L CNN
-F 1 "500u" H 8965 6605 50  0000 L CNN
+F 1 "6.8u" H 8965 6605 50  0000 L CNN
 F 2 "Capacitor_SMD:C_0805_2012Metric" H 8888 6500 50  0001 C CNN
 F 3 "~" H 8850 6650 50  0001 C CNN
@@
 P 8850 7450
 F 0 "C6" H 8965 7496 50  0000 L CNN
-F 1 "500u" H 8965 7405 50  0000 L CNN
+F 1 "6.8u" H 8965 7405 50  0000 L CNN
 F 2 "Capacitor_SMD:C_0805_2012Metric" H 8888 7300 50  0001 C CNN
 F 3 "~" H 8850 7450 50  0001 C CNN
@@
 P 8850 8250
 F 0 "C7" H 8965 8296 50  0000 L CNN
-F 1 "500u" H 8965 8205 50  0000 L CNN
+F 1 "6.8u" H 8965 8205 50  0000 L CNN
 F 2 "Capacitor_SMD:C_0805_2012Metric" H 8888 8100 50  0001 C CNN
 F 3 "~" H 8850 8250 50  0001 C CNN
@@
 P 8850 10650
 F 0 "C10" H 8965 10696 50  0000 L CNN
-F 1 "500u" H 8965 10605 50  0000 L CNN
+F 1 "6.8u" H 8965 10605 50  0000 L CNN
 F 2 "Capacitor_SMD:C_0805_2012Metric" H 8888 10500 50  0001 C CNN
 F 3 "~" H 8850 10650 50  0001 C CNN
@@
 P 8850 9850
 F 0 "C9" H 8965 9896 50  0000 L CNN
-F 1 "500u" H 8965 9805 50  0000 L CNN
+F 1 "6.8u" H 8965 9805 50  0000 L CNN
 F 2 "Capacitor_SMD:C_0805_2012Metric" H 8888 9700 50  0001 C CNN
 F 3 "~" H 8850 9850 50  0001 C CNN
@@
 P 8850 9050
 F 0 "C8" H 8965 9096 50  0000 L CNN
-F 1 "500u" H 8965 9005 50  0000 L CNN
+F 1 "6.8u" H 8965 9005 50  0000 L CNN
 F 2 "Capacitor_SMD:C_0805_2012Metric" H 8888 8900 50  0001 C CNN
 F 3 "~" H 8850 9050 50  0001 C CNN
@@
 $EndComp
 $Comp
-L power:GNDREF #PWR0118
-U 1 1 60A3CE62
-P 18150 11200
-F 0 "#PWR0118" H 18150 10950 50  0001 C CNN
-F 1 "GNDREF" H 18155 11027 50  0000 C CNN
-F 2 "" H 18150 11200 50  0001 C CNN
-F 3 "" H 18150 11200 50  0001 C CNN
-	1    18150 11200
-	1    0    0    -1
-$EndComp
-$Comp
-L power:GNDREF #PWR0119
-U 1 1 60A7BEF3
-P 18150 9050
-F 0 "#PWR0119" H 18150 8800 50  0001 C CNN
-F 1 "GNDREF" H 18155 8877 50  0000 C CNN
-F 2 "" H 18150 9050 50  0001 C CNN
-F 3 "" H 18150 9050 50  0001 C CNN
-	1    18150 9050
-	1    0    0    -1
-$EndComp
-$Comp
 L power:PWR_FLAG #FLG0114
 U 1 1 60ABAE30
@@
 P 14240 4270
 F 0 "LOGO1" H 14240 4420 50  0001 C CNN
-F 1 "Logo_Placeholder" H 14380 4270 50  0000 L CNN
+F 1 "Hallock" H 14380 4270 50  0000 L CNN
 F 2 "UTSVT_Special:Hallock_Image" H 14240 4345 50  0001 C CNN
 F 3 "" H 14240 4345 50  0001 C CNN
@@
 L utsvt-misc:Logo_Placeholder LOGO2
 U 1 1 5FC4C570
-P 14500 3700
-F 0 "LOGO2" H 14500 3850 50  0001 C CNN
-F 1 "Logo_Placeholder" H 14640 3700 50  0000 L CNN
-F 2 "UTSVT_Special:UTSVT_Logo_Symbol" H 14500 3775 50  0001 C CNN
-F 3 "" H 14500 3775 50  0001 C CNN
-	1    14500 3700
-	1    0    0    -1
-$EndComp
-$Comp
-L utsvt-misc:Logo_Placeholder LOGO3
-U 1 1 5FC56913
-P 14070 3950
-F 0 "LOGO3" H 14070 4100 50  0001 C CNN
-F 1 "Logo_Placeholder" H 14210 3950 50  0000 L CNN
-F 2 "UTSVT_Special:Aro" H 14070 4025 50  0001 C CNN
-F 3 "" H 14070 4025 50  0001 C CNN
-	1    14070 3950
+P 14200 4000
+F 0 "LOGO2" H 14200 4150 50  0001 C CNN
+F 1 "UTSVT_Logo" H 14340 4000 50  0000 L CNN
+F 2 "UTSVT_Special:UTSVT_Logo_Symbol" H 14200 4075 50  0001 C CNN
+F 3 "" H 14200 4075 50  0001 C CNN
+	1    14200 4000
 	1    0    0    -1
 $EndComp
@@
 	1    0    0    -1
 $EndComp
+Wire Wire Line
+	16800 11650 16000 11650
+Wire Wire Line
+	16800 11650 16800 11850
+Wire Wire Line
+	16000 11650 16000 11500
+NoConn ~ 16600 11700
+Connection ~ 16800 11650
+Wire Wire Line
+	16800 9450 16000 9450
+Wire Wire Line
+	16800 9450 16800 9700
+Wire Wire Line
+	16000 9450 16000 9350
+NoConn ~ 16600 9550
+Connection ~ 16800 9450
 $EndSCHEMATC

Commit message: Redoes layout to make the board smaller
Parts:
- J23, J24: footprint Connector_Molex:Molex_Micro-Fit_3.0_43650-0700_1x07_P3.00mm_Horizontal -> UTSVT_Connectors:Molex_MicroFit_01x07_Horizontal
- J25, J26: footprint Connector:Banana_Jack_1Pin -> UTSVT_Connectors:Banana_Jack_1_Pin_4mm
- TP1, TP10, TP11, TP12, TP17, TP18, TP19, TP2, TP20, TP21, TP22, TP23, TP24, TP25, TP26, TP27, TP28, TP29, TP3, TP30, TP31, TP32, TP33, TP34, TP35, TP36, TP37, TP38, TP4, TP5, TP6, TP7, TP8, TP9: footprint TestPoint:TestPoint_Keystone_5005-5009_Compact -> TestPoint:TestPoint_Pad_2.0x2.0mm
- TP13, TP14, TP15, TP16: footprint TestPoint:TestPoint_Keystone_5005-5009_Compact -> TestPoint:TestPoint_Pad_D2.0mm
Connections:
- net at J23.1 (Pin_1), TP7.1: now also J6.1 (Pin_1), J7.2 (Pin_2); no longer J6.2 (Pin_2), J7.1 (Pin_1)
- net at J23.2 (Pin_2), TP6.1: now also J5.1 (Pin_1), J6.2 (Pin_2); no longer J5.2 (Pin_2), J6.1 (Pin_1)
- net at J23.3 (Pin_3), TP5.1: now also J4.1 (Pin_1), J5.2 (Pin_2); no longer J4.2 (Pin_2), J5.1 (Pin_1)
- net at J23.4 (Pin_4), TP4.1: now also J3.1 (Pin_1), J4.2 (Pin_2); no longer J3.2 (Pin_2), J4.1 (Pin_1)
- net at J23.5 (Pin_5), TP3.1: now also J2.1 (Pin_1), J3.2 (Pin_2); no longer J2.2 (Pin_2), J3.1 (Pin_1)
- net at J23.6 (Pin_6), TP2.1: now also J1.1 (Pin_1), J2.2 (Pin_2); no longer J1.2 (Pin_2), J2.1 (Pin_1)
- net at J23.7 (Pin_7), TP1.1: now also J1.2 (Pin_2); no longer J1.1 (Pin_1)
- net at J24.3 (Pin_3), TP12.1: now also J11.1 (Pin_1); no longer J11.2 (Pin_2)
- net at J24.4 (Pin_4), TP11.1: now also J10.1 (Pin_1), J11.2 (Pin_2); no longer J10.2 (Pin_2), J11.1 (Pin_1)
- net at J24.5 (Pin_5), TP10.1: now also J10.2 (Pin_2), J9.1 (Pin_1); no longer J10.1 (Pin_1), J9.2 (Pin_2)
- net at J24.6 (Pin_6), TP9.1: now also J8.1 (Pin_1), J9.2 (Pin_2); no longer J8.2 (Pin_2), J9.1 (Pin_1)
- net at J24.7 (Pin_7), TP8.1: now also J7.1 (Pin_1), J8.2 (Pin_2); no longer J7.2 (Pin_2), J8.1 (Pin_1)
Other:
- moved on the sheet: C1, C10, C11, C12, C13, C14, C15, C2, C3, C4, C5, C6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
