File: BPS-Test.sch (KiCad schematic (older format))
At the start: 128 parts, among them J1 Conn_01x02, J10 Conn_01x02, J11 Conn_01x02, J12 Conn_01x02, J13 Conn_01x02, J14 Conn_01x02, J15 Conn_01x02, J16 Conn_01x02, J17 Conn_01x02, J18 Conn_01x02, J19 Conn_01x02, J2 Conn_01x02, J20 Conn_01x02, J21 Conn_01x02, J22 Conn_01x02, J23 Conn_01x07, J24 Conn_01x07, J25 Conn_01x01, J26 Conn_01x01, J3 Conn_01x02, J4 Conn_01x02, J5 Conn_01x02, J6 Conn_01x02, J7 Conn_01x02, J8 Conn_01x02, J9 Conn_01x02, T1 Transformer_1P_1S, T2 Transformer_1P_1S, U1 LM5180QNGURQ1, U2 LM5180QNGURQ1

Commit message: Simplifies variable circuitry and adds gerbers
Parts:
- removed C12: 22n, Capacitor_SMD:C_0805_2012Metric, symbol Device:C
- removed C13, C14: 500u, Capacitor_SMD:C_0805_2012Metric, symbol Device:C
- removed C15: 460u, Capacitor_SMD:C_0805_2012Metric, symbol Device:C
- removed D1, D2: D_Zener, Diode_SMD:D_0805_2012Metric, symbol Device:D_Zener
- removed D3, D4: D, Diode_SMD:D_0805_2012Metric, symbol Device:D
- removed D5, D6: D_Schottky, Diode_SMD:D_0805_2012Metric, symbol Device:D_Schottky
- removed R1, R3: 536k, Resistor_SMD:R_0805_2012Metric, symbol Device:R
- removed R2, R4: 100k, Resistor_SMD:R_0805_2012Metric, symbol Device:R
- removed R25, R26: 1k, Resistor_SMD:R_0805_2012Metric, symbol Device:R
- removed R5, R6: 12.1k, Resistor_SMD:R_0805_2012Metric, symbol Device:R
- removed T1, T2: Transformer_1P_1S, UTSVT_Power:transformer_wuerth_750318463, symbol Device:Transformer_1P_1S
- removed TP13: Pot1-TestPoint1, TestPoint:TestPoint_Pad_D2.0mm, symbol Connector:TestPoint
- removed TP14: Pot1-TestPoint2, TestPoint:TestPoint_Pad_D2.0mm, symbol Connector:TestPoint
- removed TP15: Pot2-TestPoint1, TestPoint:TestPoint_Pad_D2.0mm, symbol Connector:TestPoint
- removed TP16: Pot2-TestPoint2, TestPoint:TestPoint_Pad_D2.0mm, symbol Connector:TestPoint
- removed U1, U2: LM5180QNGURQ1, UTSVT_Power:SON80P400X400X80-9N, symbol utsvt-power-regulators:LM5180QNGURQ1
- added PS10, PS11: RFM-0505S, UTSVT_Power:RFM0505S, symbol utsvt-power-regulators:RFM-0505S
- added RV3, RV4: R_POT, Potentiometer_THT:Potentiometer_Piher_PT-6-V_Vertical_Hole, symbol Device:R_POT
- C1: value 460u -> 6.8u
- C11: value 22n -> 6.8u
- R10, R11, R12, R14, R15, R7, R8, R9: value 280 -> 1.4K
- R16, R17, R18, R19, R20, R21, R22, R23, R24: value 720 -> 3.6K
- RV1, RV2: footprint Potentiometer_THT:Potentiometer_Piher_PT-10-V10_Vertical -> Potentiometer_THT:Potentiometer_Piher_PT-6-V_Vertical_Hole
Connections:
- wire segments 320 -> 269
- no-connect marks 8 -> 6
Other:
- moved on the sheet: J12, J13, J14, J15, J16, J17, J18, J19, J20, J21, J22, RV1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
